File: 18650_UPS_PCB/18650_UPS_PCB.sch (KiCad schematic (older format))
At the start: 45 parts, among them J1 USB_B_Micro, J2 Conn_01x02, J3 Conn_01x02, SW1 SW_SPST, SW2 SW_SPST, SW3 SW_SPST, SW4 SW_SPST, U1 STLINK-V3MINI, U10 LR9102G-xx, U11 MP2667, U2 INA237, U5 STM32L151RCTx

Commit message: changed back to 5-way-tactile
Parts:
- removed SW1, SW2, SW3, SW4: SW_SPST, CUSTOM_FOOTPRINTS:PTS815, symbol Switch:SW_SPST
- added S1: TM-2027, CUSTOM_FOOTPRINTS:TM-2027, symbol CUSTOM_PARTS:TM-2027
Connections:
- net GND: now also S1.4 (Common)
- net MP-INT: now also U5.37 (PC6), S1.6 (Center); no longer U5.38 (PC7)
- net SW-A: now also S1.1 (A)
- net SW-B: now also S1.2 (B)
- net SW-C: now also S1.3 (C)
- net SW-D: now reaches U5.33 (PB12)
- net SW-D: now also S1.5 (D)
- no-connect marks 49 -> 48
Changed lines of the file:
@@
 	1    0    0    -1
 $EndComp
-Text GLabel 13150 4450 0    50   Input ~ 0
+Text GLabel 13150 4350 0    50   Input ~ 0
 MP-INT
 Text GLabel 14700 4450 2    50   Input ~ 0
@@
 	14600 5050 14700 5050
 Wire Wire Line
-	14700 4950 14600 4950
-Wire Wire Line
-	13150 4450 13300 4450
+	13150 4350 13300 4350
 Wire Wire Line
 	14600 3050 14750 3050
@@
 Connection ~ 2000 1550
 Wire Wire Line
-	5800 7500 5800 7700
-Wire Wire Line
-	5950 7500 5800 7500
-Wire Wire Line
-	6500 7500 6350 7500
-$Comp
-L Switch:SW_SPST SW1
-U 1 1 61345DF7
-P 6150 7500
-F 0 "SW1" H 6150 7735 50  0000 C CNN
-F 1 "SW_SPST" H 6150 7644 50  0000 C CNN
-F 2 "CUSTOM_FOOTPRINTS:PTS815" H 6150 7500 50  0001 C CNN
-F 3 "~" H 6150 7500 50  0001 C CNN
-	1    6150 7500
-	1    0    0    -1
-$EndComp
-$Comp
-L power:GND #PWR0124
-U 1 1 61596BD9
-P 5800 7700
-F 0 "#PWR0124" H 5800 7450 50  0001 C CNN
-F 1 "GND" H 5805 7527 50  0000 C CNN
-F 2 "" H 5800 7700 50  0001 C CNN
-F 3 "" H 5800 7700 50  0001 C CNN
-	1    5800 7700
-	1    0    0    -1
-$EndComp
-Text GLabel 6500 7500 2    50   Input ~ 0
-MP-INT
-Wire Wire Line
 	14700 2750 14600 2750
 Wire Wire Line
 	13200 3750 13300 3750
-$Comp
-L power:GND #PWR0119
-U 1 1 6111C509
-P 3900 7000
-F 0 "#PWR0119" H 3900 6750 50  0001 C CNN
-F 1 "GND" H 3905 6827 50  0000 C CNN
-F 2 "" H 3900 7000 50  0001 C CNN
-F 3 "" H 3900 7000 50  0001 C CNN
-	1    3900 7000
-	1    0    0    -1
-$EndComp
-Wire Wire Line
-	3900 7000 3900 6800
-Wire Wire Line
-	3900 6800 4000 6800
-Text GLabel 4550 6800 2    50   Input ~ 0
+Text GLabel 5150 6600 1    50   Input ~ 0
 SW-A
 Wire Wire Line
-	4400 6800 4550 6800
-$Comp
-L Switch:SW_SPST SW2
-U 1 1 61154FD9
-P 4200 6800
-F 0 "SW2" H 4200 7035 50  0000 C CNN
-F 1 "SW_SPST" H 4200 6944 50  0000 C CNN
-F 2 "CUSTOM_FOOTPRINTS:PTS815" H 4200 6800 50  0001 C CNN
-F 3 "~" H 4200 6800 50  0001 C CNN
-	1    4200 6800
-	1    0    0    -1
-$EndComp
-$Comp
-L power:GND #PWR0120
-U 1 1 6118A3A3
-P 3900 7750
-F 0 "#PWR0120" H 3900 7500 50  0001 C CNN
-F 1 "GND" H 3905 7577 50  0000 C CNN
-F 2 "" H 3900 7750 50  0001 C CNN
-F 3 "" H 3900 7750 50  0001 C CNN
-	1    3900 7750
-	1    0    0    -1
-$EndComp
-Wire Wire Line
-	3900 7750 3900 7550
-Wire Wire Line
-	3900 7550 4000 7550
-Text GLabel 4550 7550 2    50   Input ~ 0
+	5150 6750 5150 6600
+Text GLabel 4550 7050 0    50   Input ~ 0
 SW-B
 Wire Wire Line
-	4400 7550 4550 7550
-$Comp
-L Switch:SW_SPST SW3
-U 1 1 6118A3AD
-P 4200 7550
-F 0 "SW3" H 4200 7785 50  0000 C CNN
-F 1 "SW_SPST" H 4200 7694 50  0000 C CNN
-F 2 "CUSTOM_FOOTPRINTS:PTS815" H 4200 7550 50  0001 C CNN
-F 3 "~" H 4200 7550 50  0001 C CNN
-	1    4200 7550
-	1    0    0    -1
-$EndComp
-$Comp
-L power:GND #PWR0121
-U 1 1 61197B26
-P 5800 7000
-F 0 "#PWR0121" H 5800 6750 50  0001 C CNN
-F 1 "GND" H 5805 6827 50  0000 C CNN
-F 2 "" H 5800 7000 50  0001 C CNN
-F 3 "" H 5800 7000 50  0001 C CNN
-	1    5800 7000
-	1    0    0    -1
-$EndComp
-Wire Wire Line
-	5800 7000 5800 6800
-Wire Wire Line
-	5800 6800 5900 6800
-Text GLabel 6450 6800 2    50   Input ~ 0
+	4700 7050 4550 7050
+Text GLabel 5150 7700 3    50   Input ~ 0
 SW-C
 Wire Wire Line
-	6300 6800 6450 6800
-$Comp
-L Switch:SW_SPST SW4
-U 1 1 61197B30
-P 6100 6800
-F 0 "SW4" H 6100 7035 50  0000 C CNN
-F 1 "SW_SPST" H 6100 6944 50  0000 C CNN
-F 2 "CUSTOM_FOOTPRINTS:PTS815" H 6100 6800 50  0001 C CNN
-F 3 "~" H 6100 6800 50  0001 C CNN
-	1    6100 6800
-	1    0    0    -1
-$EndComp
+	5150 7550 5150 7700
 Text GLabel 14700 5250 2    50   Input ~ 0
 SW-A
@@
 Text GLabel 14700 5050 2    50   Input ~ 0
 SW-C
-NoConn ~ 13200 4350
-Wire Wire Line
-	13200 4350 13300 4350
-NoConn ~ 14700 4950
+NoConn ~ 13200 4450
+Wire Wire Line
+	13200 4450 13300 4450
+$Comp
+L CUSTOM_PARTS:TM-2027 S1
+U 1 1 61148628
+P 5050 6800
+F 0 "S1" H 5300 6850 50  0000 C CNN
+F 1 "TM-2027" H 4800 6850 50  0000 C CNN
+F 2 "CUSTOM_FOOTPRINTS:TM-2027" H 5900 6950 50  0001 C CNN
+F 3 "" H 5400 6800 50  0001 C CNN
+	1    5050 6800
+	1    0    0    -1
+$EndComp
+$Comp
+L power:GND #PWR0119
+U 1 1 61148C56
+P 4550 7350
+F 0 "#PWR0119" H 4550 7100 50  0001 C CNN
+F 1 "GND" H 4555 7177 50  0000 C CNN
+F 2 "" H 4550 7350 50  0001 C CNN
+F 3 "" H 4550 7350 50  0001 C CNN
+	1    4550 7350
+	1    0    0    -1
+$EndComp
+Wire Wire Line
+	4550 7350 4550 7250
+Wire Wire Line
+	4550 7250 4700 7250
+Text GLabel 5750 7050 2    50   Input ~ 0
+SW-D
+Wire Wire Line
+	5600 7050 5750 7050
+Wire Wire Line
+	5750 7250 5600 7250
+Text GLabel 5750 7250 2    50   Input ~ 0
+MP-INT
+Text GLabel 14700 4950 2    50   Input ~ 0
+SW-D
+Wire Wire Line
+	14700 4950 14600 4950
 $EndSCHEMATC
